Commit message: 2nd round of more expirimental nav2-fixes

File: perception/config/phone_mount.urdf (robot description, URDF)
Before this commit: robot couch_phone_mount, 4 links, 3 joints
Joints:
- joint base_to_phone_mount: origin xyz=0 0 1.5 rpy=3.141592653589793 -1.5707963267948966 0 -> xyz=0 0 1.5 rpy=0 0 0
